File: esp32s3board.kicad_pcb (KiCad board)
At the start: 2 copper layers, 53.3 x 57.2 mm, 49 parts, among them J1 Arduino_UNO_R3, J2 USB_C_Receptacle_USB2.0_14P, J3 HOST, J4 Power, J5 EN, J6 BOOT, J7 JTAG_SEL, J8 ZUSI, Q1 BC847BDW1, SW1 RESET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

Commit message: Switch to horizontal pin headers
Parts:
- removed the J3 at (80.0, 44.2)
- added JP1: SolderJumper_2_Open, Jumper:SolderJumper-2_P1.3mm_Open_Pad1.0x1.5mm, B.Cu at (80.0, 44.3)
- J3: renamed from J4; footprint Connector_PinHeader_2.54mm:PinHeader_1x02_P2.54mm_Vertical -> Connector_PinHeader_2.54mm:PinHeader_1x02_P2.54mm_Horizontal
- J4: renamed from J5; value EN -> PROG; footprint Connector_PinHeader_2.54mm:PinHeader_1x02_P2.54mm_Vertical -> Connector_PinHeader_2.54mm:PinHeader_1x02_P2.54mm_Horizontal
- J5: renamed from J6; value BOOT -> RESET; footprint Connector_PinHeader_2.54mm:PinHeader_1x02_P2.54mm_Vertical -> Connector_PinHeader_2.54mm:PinHeader_1x02_P2.54mm_Horizontal
- J6: renamed from J7; value JTAG_SEL -> CONFIG; footprint Connector_PinHeader_2.54mm:PinHeader_1x02_P2.54mm_Vertical -> Connector_PinHeader_2.54mm:PinHeader_1x02_P2.54mm_Horizontal
- moved J6 7.87 mm to (109.1, 56.9), turned to -90 degrees
- moved C1 6.36 mm to (94.2, 36.3)
- moved C2 5.85 mm to (94.2, 40.4), turned to -90 degrees
- moved R8 5.62 mm to (94.2, 38.4), turned to -90 degrees
- moved R7 3.92 mm to (104.1, 55.9), turned to 90 degrees
- moved R4 3.03 mm to (94.2, 42.4), turned to 90 degrees
- moved J4 2.55 mm to (96.8, 38.7), turned to 90 degrees
- moved J5 2.54 mm to (122.7, 56.9), turned to -90 degrees
- moved J3 2.42 mm to (105.9, 87.5), turned to -90 degrees
- renumbered J8 to J7
Routing:
- net +3V3: track 111.8 -> 117.6 mm
- net VIN: track 73.5 -> 76.1 mm
- net GND: track 19.8 -> 18.5 mm
- net ZUSI_DATA: track 26.2 -> 25.2 mm
- net D8: track 16.7 -> 15.7 mm
- net EN: track 95.4 -> 96.3 mm
- net BOOT: track 25.2 -> 26.0 mm
- net +5V: track 70.5 -> 69.7 mm
- net Net-(D1-TVS4): track 24.3 -> 23.5 mm, vias 0 -> 1
- net JTAG_SEL: track 6.66 -> 7.31 mm, vias 0 -> 1
- net ZUSI_CLK: track 25.2 -> 24.6 mm
- net D2: track 36.2 -> 36.8 mm
Other:
- board text removed: "BOOT"
- board text removed: "EN"
