File: esp32s3board.kicad_sch (KiCad schematic)
At the start: 45 parts, among them J1 Arduino_UNO_R3, J2 USB_C_Receptacle_USB2.0_14P, J3 HOST, J4 Power, J5 EN, J6 BOOT, J7 JTAG_SEL, J8 ZUSI, Q1 BC847BDW1, SW1 RESET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

Commit message: Switch to horizontal pin headers
Parts:
- removed J3: HOST, Connector_PinHeader_2.54mm:PinHeader_1x02_P2.54mm_Vertical, symbol Connector_Generic:Conn_01x02
- added JP1: SolderJumper_2_Open, Jumper:SolderJumper-2_P1.3mm_Open_Pad1.0x1.5mm, symbol Jumper:SolderJumper_2_Open
- J3: renamed from J4; footprint Connector_PinHeader_2.54mm:PinHeader_1x02_P2.54mm_Vertical -> Connector_PinHeader_2.54mm:PinHeader_1x02_P2.54mm_Horizontal
- J4: renamed from J5; value EN -> PROG; footprint Connector_PinHeader_2.54mm:PinHeader_1x02_P2.54mm_Vertical -> Connector_PinHeader_2.54mm:PinHeader_1x02_P2.54mm_Horizontal
- J5: renamed from J6; value BOOT -> RESET; footprint Connector_PinHeader_2.54mm:PinHeader_1x02_P2.54mm_Vertical -> Connector_PinHeader_2.54mm:PinHeader_1x02_P2.54mm_Horizontal
- J6: renamed from J7; value JTAG_SEL -> CONFIG; footprint Connector_PinHeader_2.54mm:PinHeader_1x02_P2.54mm_Vertical -> Connector_PinHeader_2.54mm:PinHeader_1x02_P2.54mm_Horizontal
- renumbered J8 to J7
Connections:
- net +5V: now also JP1.2 (B)
- net at D1.6 (TVS4), J2.A4 (VBUS), J2.A9 (VBUS)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: now also JP1.1 (A)
Changed lines of the file:
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@@
     (stroke (width 0) (type default))
   )
-  (wire (pts (xy 111.125 140.97) (xy 111.125 143.51))
-    (stroke (width 0) (type default))
-  )
   (wire (pts (xy 41.275 187.96) (xy 41.275 189.23))
     (stroke (width 0) (type default))
@@
     (stroke (width 0) (type default))
   )
-  (wire (pts (xy 112.395 140.97) (xy 111.125 140.97))
-    (stroke (width 0) (type default))
-  )
   (wire (pts (xy 240.665 146.685) (xy 240.665 145.415))
     (stroke (width 0) (type default))
@@
     (stroke (width 0) (type default))
   )
+  (wire (pts (xy 111.125 133.35) (xy 111.125 134.62))
+    (stroke (width 0) (type default))
+  )
   (wire (pts (xy 123.19 95.885) (xy 124.46 95.885))
     (stroke (width 0) (type default))
@@
     (stroke (width 0) (type default))
   )
-  (wire (pts (xy 111.125 138.43) (xy 112.395 138.43))
-    (stroke (width 0) (type default))
-  )
   (wire (pts (xy 46.355 134.62) (xy 46.355 133.985))
     (stroke (width 0) (type default))
@@
     (stroke (width 0) (type default))
   )
-  (wire (pts (xy 111.125 137.16) (xy 111.125 138.43))
-    (stroke (width 0) (type default))
-  )
   (wire (pts (xy 161.925 75.565) (xy 161.925 76.835))
     (stroke (width 0) (type default))
@@
     (stroke (width 0) (type default))
   )
+  (wire (pts (xy 111.125 142.24) (xy 111.125 143.51))
+    (stroke (width 0) (type default))
+  )
   (wire (pts (xy 97.155 162.56) (xy 100.965 162.56))
     (stroke (width 0) (type default))
@@
   (symbol (lib_id "Connector_Generic:Conn_01x02") (at 152.4 140.335 0) (mirror y) (unit 1)
     (in_bom yes) (on_board yes) (dnp no)
-    (property "Reference" "J4" (at 152.4 137.795 0)
+    (property "Reference" "J3" (at 152.4 137.795 0)
       (effects (font (size 1.27 1.27)))
     )
@@
       (effects (font (size 1.27 1.27)))
     )
-    (property "Footprint" "Connector_PinHeader_2.54mm:PinHeader_1x02_P2.54mm_Vertical" (at 152.4 140.335 0)
+    (property "Footprint" "Connector_PinHeader_2.54mm:PinHeader_1x02_P2.54mm_Horizontal" (at 152.4 140.335 0)
       (effects (font (size 1.27 1.27)) hide)
     )
@@
       (project "esp32s3board"
         (path "/41e00285-a902-4fec-b014-18776c0aad20"
-          (reference "J4") (unit 1)
+          (reference "J3") (unit 1)
         )
       )
@@
   (symbol (lib_id "Connector_Generic:Conn_01x04") (at 262.255 41.275 0) (unit 1)
     (in_bom yes) (on_board yes) (dnp no)
-    (property "Reference" "J8" (at 260.985 36.195 0)
+    (property "Reference" "J7" (at 260.985 36.195 0)
       (effects (font (size 1.27 1.27)) (justify left))
     )
@@
       (project "esp32s3board"
         (path "/41e00285-a902-4fec-b014-18776c0aad20"
-          (reference "J8") (unit 1)
+          (reference "J7") (unit 1)
         )
       )
@@
     )
   )
-  (symbol (lib_id "power:+5V") (at 111.125 137.16 0) (unit 1)
+  (symbol (lib_id "power:+5V") (at 111.125 133.35 0) (unit 1)
     (in_bom yes) (on_board yes) (dnp no)
-    (property "Reference" "#PWR011" (at 111.125 140.97 0)
+    (property "Reference" "#PWR011" (at 111.125 137.16 0)
       (effects (font (size 1.27 1.27)) hide)
     )
-    (property "Value" "+5V" (at 111.125 133.35 0)
+    (property "Value" "+5V" (at 111.125 129.54 0)
       (effects (font (size 1.27 1.27)))
     )
-    (property "Footprint" "" (at 111.125 137.16 0)
+    (property "Footprint" "" (at 111.125 133.35 0)
       (effects (font (size 1.27 1.27)) hide)
     )
-    (property "Datasheet" "" (at 111.125 137.16 0)
+    (property "Datasheet" "" (at 111.125 133.35 0)
       (effects (font (size 1.27 1.27)) hide)
     )
@@
   (symbol (lib_id "Connector_Generic:Conn_01x02") (at 155.575 109.855 0) (mirror y) (unit 1)
     (in_bom yes) (on_board yes) (dnp no)
-    (property "Reference" "J7" (at 155.575 107.315 0)
+    (property "Reference" "J6" (at 155.575 107.315 0)
       (effects (font (size 1.27 1.27)))
     )
-    (property "Value" "JTAG_SEL" (at 155.575 114.935 0)
+    (property "Value" "CONFIG" (at 155.575 114.935 0)
       (effects (font (size 1.27 1.27)))
     )
-    (property "Footprint" "Connector_PinHeader_2.54mm:PinHeader_1x02_P2.54mm_Vertical" (at 155.575 109.855 0)
+    (property "Footprint" "Connector_PinHeader_2.54mm:PinHeader_1x02_P2.54mm_Horizontal" (at 155.575 109.855 0)
       (effects (font (size 1.27 1.27)) hide)
     )
@@
       (project "esp32s3board"
         (path "/41e00285-a902-4fec-b014-18776c0aad20"
-          (reference "J7") (unit 1)
+          (reference "J6") (unit 1)
         )
       )
@@
     )
   )
+  (symbol (lib_id "Jumper:SolderJumper_2_Open") (at 111.125 138.43 90) (unit 1)
+    (in_bom yes) (on_board yes) (dnp no) (fields_autoplaced)
+    (property "Reference" "JP1" (at 113.665 137.16 90)
+      (effects (font (size 1.27 1.27)) (justify right))
+    )
+    (property "Value" "SolderJumper_2_Open" (at 113.665 139.7 90)
+      (effects (font (size 1.27 1.27)) (justify right) hide)
+    )
+    (property "Footprint" "Jumper:SolderJumper-2_P1.3mm_Open_Pad1.0x1.5mm" (at 111.125 138.43 0)
+      (effects (font (size 1.27 1.27)) hide)
+    )
+    (property "Datasheet" "~" (at 111.125 138.43 0)
+      (effects (font (size 1.27 1.27)) hide)
+    )
+    (pin "2")
+    (pin "1")
+    (instances
+      (project "esp32s3board"
+        (path "/41e00285-a902-4fec-b014-18776c0aad20"
+          (reference "JP1") (unit 1)
+        )
+      )
+    )
+  )
   (symbol (lib_id "Device:C_Small") (at 275.59 142.875 0) (unit 1)
     (in_bom yes) (on_board yes) (dnp no)
@@
     )
   )
-  (symbol (lib_id "Connector_Generic:Conn_01x02") (at 117.475 138.43 0) (unit 1)
-    (in_bom yes) (on_board yes) (dnp no) (fields_autoplaced)
-    (property "Reference" "J3" (at 120.015 138.43 0)
-      (effects (font (size 1.27 1.27)) (justify left))
-    )
-    (property "Value" "HOST" (at 120.015 140.97 0)
-      (effects (font (size 1.27 1.27)) (justify left))
-    )
-    (property "Footprint" "Connector_PinHeader_2.54mm:PinHeader_1x02_P2.54mm_Vertical" (at 117.475 138.43 0)
-      (effects (font (size 1.27 1.27)) hide)
-    )
-    (property "Datasheet" "~" (at 117.475 138.43 0)
-      (effects (font (size 1.27 1.27)) hide)
-    )
-    (pin "1")
-    (pin "2")
-    (instances
-      (project "esp32s3board"
-        (path "/41e00285-a902-4fec-b014-18776c0aad20"
-          (reference "J3") (unit 1)
-        )
-      )
-    )
-  )
   (symbol (lib_id "Device:C_Small") (at 240.665 142.875 0) (unit 1)
     (in_bom yes) (on_board yes) (dnp no) (fields_autoplaced)
@@
   (symbol (lib_id "Connector_Generic:Conn_01x02") (at 155.575 73.025 0) (mirror y) (unit 1)
     (in_bom yes) (on_board yes) (dnp no)
-    (property "Reference" "J6" (at 155.575 70.485 0)
+    (property "Reference" "J5" (at 155.575 70.485 0)
       (effects (font (size 1.27 1.27)))
     )
-    (property "Value" "BOOT" (at 155.575 78.105 0)
+    (property "Value" "RESET" (at 155.575 78.105 0)
       (effects (font (size 1.27 1.27)))
     )
-    (property "Footprint" "Connector_PinHeader_2.54mm:PinHeader_1x02_P2.54mm_Vertical" (at 155.575 73.025 0)
+    (property "Footprint" "Connector_PinHeader_2.54mm:PinHeader_1x02_P2.54mm_Horizontal" (at 155.575 73.025 0)
       (effects (font (size 1.27 1.27)) hide)
     )
@@
       (project "esp32s3board"
         (path "/41e00285-a902-4fec-b014-18776c0aad20"
-          (reference "J6") (unit 1)
+          (reference "J5") (unit 1)
         )
       )
@@
   (symbol (lib_id "Connector_Generic:Conn_01x02") (at 155.575 39.37 0) (mirror y) (unit 1)
     (in_bom yes) (on_board yes) (dnp no)
-    (property "Reference" "J5" (at 155.575 36.83 0)
+    (property "Reference" "J4" (at 155.575 36.83 0)
       (effects (font (size 1.27 1.27)))
     )
-    (property "Value" "EN" (at 155.575 44.45 0)
+    (property "Value" "PROG" (at 155.575 44.45 0)
       (effects (font (size 1.27 1.27)))
     )
-    (property "Footprint" "Connector_PinHeader_2.54mm:PinHeader_1x02_P2.54mm_Vertical" (at 155.575 39.37 0)
+    (property "Footprint" "Connector_PinHeader_2.54mm:PinHeader_1x02_P2.54mm_Horizontal" (at 155.575 39.37 0)
       (effects (font (size 1.27 1.27)) hide)
     )
@@
       (project "esp32s3board"
         (path "/41e00285-a902-4fec-b014-18776c0aad20"
-          (reference "J5") (unit 1)
+          (reference "J4") (unit 1)
         )
       )
